Commit message: - benchmarkConfig.m (neu):	Enthält alle Zahlen, die ein Experiment beeinflussen: Trajektorie, Masse der Basis (25 kg), Reward-Gewichte (200/8 usw.), τ_max, d_safe, Startpose, Seed. Einzelwerte lassen sich überschreiben, z. B. benchmarkConfig('reward.wori', 400).
- setupSpaceRobotEnv.m:	Übernimmt alles aus der Konfiguration, beherrscht Kreis und Zwei-Segment-Bahn, liefert cfg mit zurück.

- localResetFunction.m:	Optionale zufällige Startpose q0 ± range_deg.

- parametrizeSpaceRobotModel.m (neu): SpaceRobot.slx	Masse, Trägheit, Gelenkdämpfung, Startwinkel, Momentensättigung und Reward-Gewichte werden jetzt aus dem Workspace gelesen statt fest im Modell zu stehen. Das Skript dokumentiert die Änderung, und ein zweiter Aufruf ändert nichts mehr.

- computeKPIsFromLogs.m:	K7 ist jetzt der mittlere Jerk (niedriger ist besser), wie im Paper definiert.
SpaceRobot.urdf	Trägheitsdaten an das Simscape-Modell angeglichen: Basis 25 kg und 5 kg·m², Armglieder izz = 0.1, Endeffektor ohne Masse.

File: SpaceRobot.urdf (robot description, URDF)
Before this commit: robot floating_arm, 6 links, 5 joints
Links:
- link base_link: mass 65.0 -> 25.0
- link ee_link: mass 0.1 -> None

Commit message: Stresstest-Bedingungen im Modell, Impulsmonitor und echte Gesamtmassen (A27, A42)
- Sensorrauschen auf der Beobachtung (noise.obs_std, Block "obs noise"): eigene
  Folge je Episode, in der Auswertung gleich für alle Agenten. Reward und KPIs
  sehen weiter die ungestörten Signale.
- Äußeres Gelenkmoment (dist.tau, dist.t_on/t_off, Block "joint disturbance")
  nach der Saturation. Reward, K8 und K9 sehen nur das Moment des Agenten.
- Impulsmonitor rechnet mit robotP statt fest 5 kg, p_tot wird geloggt (A27).
  Kontrolle: max |p| vorher 0,3-1,9 N s, jetzt 7e-8 bis 3e-4 N s.
- A42: Die Solid-Blöcke "Visual" aus dem URDF-Import tragen eigene Masse.
  Simuliert wurden 30 kg Basis und 2 kg je Glied, nicht 25 und 1. benchmarkConfig
  enthält jetzt die Gesamtwerte (cfg.version = 2), setupSpaceRobotEnv teilt sie
  exakt auf beide Blöcke auf, upgradeConfig rechnet alte Agentendateien um,
  URDF angeglichen. param_scale skaliert damit auch die Geometrieblöcke.
- Regressionstest: Mit Nominalkonfiguration sind KPI-Tabellen, alle geloggten
  Signale (6 Agenten x 31 Episoden) und Kurztrainings bitgleich zu benchmark_v2.

Fortschrittsanzeige je Episode und Kampagnenstatus

- progressLogger: trainOne schreibt je Trainingsepisode eine Zeile nach
  results/<Kampagne>/progress/. Der Logger speichert selbst nichts, das
  Training bleibt bitgleich.
- campaignStatus("<Kampagne>"): erfolgreiche, laufende und wartende Läufe mit
  Episodenzahl, Restzeit und Reward. Läuft auch in einer zweiten MATLAB-Sitzung.
- runCampaign: Jobs dürfen eigene Kampagne und Config tragen, dadurch mehrere
  Studien in einem Pool. Statusausgabe alle 10 Minuten.

Teil-C-Kampagnen, 10 Seeds und getrennte Auswertung von Abbruchrate und KPIs

- partCJobs/runPartC: R2.4b (PPO/TRPO/SAC mit W_ori und W_p je halbiert und
  verdoppelt), Ablation und Sensitivität des optimierten PPO, Zwei-Segment-Bahn,
  Stresstests der benchmark_v2-Agenten. Reward-Varianten werden mit den
  nominalen Gewichten ausgewertet, damit K1 vergleichbar bleibt.
- runBenchmark auf Seeds 0-9. Die Seeds 0-4 bleiben gültig, es kommen nur 5-9
  dazu. Zwei-Segment-Bahn 10 Seeds, die beschreibenden Studien 5 Seeds.
- analyzeBenchmark: Tabelle 1 mit erfolgreichen Läufen, Abbruchrate und
  Abbruchgrund über alle Läufe, Tabelle 2 mit den KPIs nur über die
  erfolgreichen Läufe. Erfolgreich heißt: keine der 31 Auswertungsepisoden
  bricht ab. Mann-Whitney auf Seed-Ebene über die erfolgreichen Läufe,
  Fisher-Test für die Abbruchraten, beides Holm-korrigiert. Ausgabe als CSV
  und LaTeX je Bedingung.

File: SpaceRobot.urdf (robot description, URDF)
Before this commit: robot floating_arm, 6 links, 5 joints
Links:
- link base_link: mass 25.0 -> 30.0
- link link1: mass 1.0 -> 2.0
- link link2: mass 1.0 -> 2.0
- link link3: mass 1.0 -> 2.0
- link link4: mass 1.0 -> 2.0
